File: kicad/Push Button Latch with USB.kicad_pcb (KiCad board)
At the start: 2 copper layers, 16 parts, among them J1 Conn_01x02, J2 Conn_01x04, J3 USB_B_Micro, Q1 SIA527DJ-T1-GE3, Q2 SIA527DJ-T1-GE3, SW1 SW_Push, U1 AMS1117-3.3

Commit message: Seems like rev.A is finished
Parts:
- added C3: 100n, Capacitor_SMD:C_0805_2012Metric, F.Cu at (51.3, 75.6)
- added C4: 10u, Capacitor_SMD:C_0805_2012Metric, F.Cu at (53.2, 75.6)
- added C5: 100n, Capacitor_SMD:C_0805_2012Metric, F.Cu at (51.3, 61.8)
- added C6: 10u, Capacitor_SMD:C_0805_2012Metric, F.Cu at (53.2, 61.8)
- added J4: Conn_01x03, Connector_PinHeader_2.54mm:PinHeader_1x03_P2.54mm_Vertical, B.Cu at (48.3, 76.2)
- added QR*****: barn53, barn53, B.Cu at (34.7, 70.5)
- added REF**: HOLE, HOLE, F.Cu at (26.9, 62.2)
- D2: value LED -> Power
- J1: value Conn_01x02 -> USB_B_Micro; footprint Connector_PinHeader_2.54mm:PinHeader_1x02_P2.54mm_Vertical -> barn53-kicad:MicroUSB_through_hole_fixing
- J2: value Conn_01x04 -> Conn_01x03; footprint Connector_PinHeader_2.54mm:PinHeader_1x04_P2.54mm_Vertical -> Connector_PinHeader_2.54mm:PinHeader_1x03_P2.54mm_Vertical; moved to B.Cu
- J3: value USB_B_Micro -> Conn_01x03; footprint barn53-kicad:MicroUSB_through_hole_fixing -> Connector_PinHeader_2.54mm:PinHeader_1x03_P2.54mm_Vertical; moved to B.Cu
- SW1: value SW_Push -> On/Off
- moved D2 68.0 mm to (34.2, 75.4), turned to 180 degrees
- moved R1 54.0 mm to (38.9, 69.1)
- moved J1 53.7 mm to (30.4, 70.9), turned to 270 degrees
- moved U1 51.0 mm to (50.5, 68.3), turned to 90 degrees
- moved J2 46.6 mm to (38.1, 61.0), turned to 90 degrees
- moved Q2 46.4 mm to (36.8, 65.5)
- moved Q1 45.1 mm to (33.7, 65.6)
- moved R2 44.7 mm to (37.7, 74.7), turned to 90 degrees
- moved J3 43.7 mm to (48.3, 61.0), turned to 90 degrees
- moved SW1 39.8 mm to (44.6, 72.6), turned to 90 degrees
- moved C1 37.1 mm to (34.4, 73.3), turned to 180 degrees
- moved R3 34.9 mm to (34.2, 69.7), turned to 90 degrees
- moved D1 33.3 mm to (28.7, 65.0), turned to 180 degrees
- moved R5 33.3 mm to (39.6, 66.0), turned to 90 degrees
- moved R4 31.7 mm to (39.6, 74.7), turned to 90 degrees
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Connections:
- C1 pad 1: Net-(C1-Pad1) -> /Bt1
- D1 pad 1: (no net) -> /VIn
- D1 pad 2: (no net) -> /VBus
- J1 pad 1: (no net) -> /VBus
- J2 pad 1: (no net) -> /Off
- J2 pad 2: (no net) -> /Bt2
- J2 pad 3: (no net) -> /Bt1
- J3 pad 1: (no net) -> GND
- J3 pad 2: (no net) -> /+3V3
- J3 pad 3: (no net) -> /VOut
- Q1 pad 6: Net-(Q1-Pad6) -> /Bt2
- Q2 pad 2: Net-(Q1-Pad6) -> /Bt2
- R2 pad 2: Net-(C1-Pad1) -> /Bt1
- R3 pad 1: Net-(Q1-Pad6) -> /Bt2
- R3 pad 6: /Off -> Net-(Q1-Pad3)
- R3 pad 7: Net-(Q1-Pad3) -> /Off
- SW1 pad 1: Net-(C1-Pad1) -> /Bt1
- SW1 pad 2: Net-(Q1-Pad6) -> /Bt2
- U1 pad 1: (no net) -> GND
- U1 pad 2: Net-(U1-Pad2) -> /+3V3
- U1 pad 3: (no net) -> /VOut
Routing:
- net /VOut: track 0.00 -> 45.0 mm, vias 0 -> 3
- net /+3V3: track 0.00 -> 35.8 mm, vias 0 -> 1
- net /Bt1: track 0.00 -> 35.2 mm, vias 0 -> 6
- net /Bt2: track 0.00 -> 30.9 mm, vias 0 -> 3
- net /Off: track 0.00 -> 24.9 mm, vias 0 -> 1
- net /VIn: track 0.00 -> 23.0 mm, vias 0 -> 3
- net Net-(Q2-Pad6): track 0.00 -> 22.3 mm
- net /VBus: track 0.00 -> 6.42 mm
- net Net-(Q1-Pad5): track 0.00 -> 5.94 mm
- net Net-(Q1-Pad3): track 0.00 -> 5.71 mm
- net Net-(D2-Pad1): track 0.00 -> 5.59 mm
- net Net-(Q2-Pad5): track 0.00 -> 2.44 mm
- net GND: vias 0 -> 2
- added copper zone on B.Cu, net GND
- added copper zone on F.Cu, net GND
Other:
- board outline added: 31.2 x 17.8 mm
- net class Default: clearance 0.2 -> 0.1524; trace_width 0.25 -> 0.254; via_dia 0.8 -> 0.5588; via_drill 0.4 -> 0.381
- net class Power added: clearance 0.1524, trace_width 0.381, via_dia 0.5588, via_drill 0.381
- rule trace_clearance: 0.2 -> 0.1524
- board text added: "3.3V"
- board text added: "5V"
- board text added: "Button"
- board text added: "GND"
- board text added: "Off"
- board text added: "barn53.de Push Button Latch with digital Off and Micro USB rev.A - 02/20"
